Commit message: main launch works but with an error on front caster wheel

File: urdf/barista_robot_model.urdf (robot description, URDF)
Before this commit: robot robot, 15 links, 14 joints
Links:
- added link laser_scan_link, mass 0.3; collision cylinder length=0.042 radius=0.038; visual mesh filename=file://$(find barista_robot_description)/meshes/rplidar_a2.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 scale=1 1 1
- link back_pitch_link: mass 0.001 -> 0.5
- link back_roll_link: mass 0.001 -> 0.5; geometry collision cylinder length=0.005 radius=0.0045000000000000005; visual cylinder length=0.005 radius=0.0045000000000000005
- link back_yaw_link: mass 0.001 -> 0.5; geometry collision cylinder length=0.005 radius=0.0045000000000000005; visual cylinder length=0.005 radius=0.0045000000000000005
- link base_link: mass 10.5 -> 5.5
- link front_pitch_link: mass 0.001 -> 0.5
- link front_roll_link: mass 0.001 -> 0.5; geometry collision cylinder length=0.005 radius=0.0045000000000000005; visual cylinder length=0.005 radius=0.0045000000000000005
- link front_yaw_link: mass 0.001 -> 0.5; geometry collision cylinder length=0.005 radius=0.0045000000000000005; visual cylinder length=0.005 radius=0.0045000000000000005
- link head: mass 5 -> 1.5
- link left_back_support_link: mass 5 -> 0.25
- link left_front_support_link: mass 5 -> 0.25
- link left_wheel: mass 5 -> 2.5
- link right_back_support_link: mass 5 -> 0.25
- link right_front_support_link: mass 5 -> 0.25
- link right_wheel: mass 5 -> 2.5
Joints:
- added joint laser_scan_link_joint: type fixed, parent base_link, child laser_scan_link, origin xyz=0.11 0 0.0925 rpy=0 0 0, axis 0 0 0
- joint head_joint: axis 0 1 0 -> (none); limit effort=10000 velocity=1000 -> (none)
- joint joint_bar_4: axis 0 1 0 -> (none); limit effort=10000 velocity=1000 -> (none)

Commit message: Part1 complete

File: urdf/barista_robot_model.urdf (robot description, URDF)
Before this commit: robot Morty, 16 links, 15 joints
Links:
- removed link base_footprint
- link back_pitch_link: geometry collision sphere radius=0.030; visual sphere radius=0.030
Joints:
- removed joint base_link_joint
