Commit message: first try

File: xacro/barista_robot_model.urdf.xacro (robot description, xacro)
@@ -1,4 +1,5 @@
 <?xml version="1.0"?>
-<robot xmlns:xacro="http://www.ros.org/wiki/xacro" name="bot">
+<robot xmlns:xacro="http://www.ros.org/wiki/xacro" name="my_robot">
+<xacro:property name="robot_name"  value="$(arg robot_name)"/>
 <xacro:include filename="$(find barista_robot_description)/xacro/wheel.xacro" />
 <xacro:include filename="$(find barista_robot_description)/xacro/standoff.xacro" />
@@ -30,4 +31,6 @@
 <xacro:property name="mesh_path"     value="file://$(find barista_robot_description)/meshes/rplidar_a2.dae"/>
 <xacro:property name="include_laser" value="false"/>
+  <link name="base_footprint">
+  </link>
 <!-- Base link  -->
     <link name="base_link">
@@ -50,4 +53,9 @@
         </inertial>
     </link>
+  <joint name="base_link_joint" type="fixed">
+    <origin rpy="0 0 0" xyz="0 0 0" />
+    <parent link="base_footprint" />
+    <child link="base_link" />
+  </joint>
   <!-- Wheel Left -->
  <xacro:wheel  wheel_name="left_wheel"        wheel_length=  "${wheel_length}"
@@ -162,6 +170,7 @@
   <!-- JOINT PUBLISHER -->
   <gazebo>
-    <plugin name="bot_joint_state" filename="libgazebo_ros_joint_state_publisher.so">
+    <plugin name="barista_joint_state" filename="libgazebo_ros_joint_state_publisher.so">
       <ros>
+          <namespace>/${robot_name}</namespace>
           <remapping>~/out:=joint_states</remapping>
       </ros>
@@ -180,18 +189,22 @@
   <gazebo>
     <plugin filename="libgazebo_ros_diff_drive.so" name="differential_drive_controller">
-      <!-- wheels -->
-      <left_joint>joint_left_wheel</left_joint>
-      <right_joint>joint_right_wheel</right_joint>
-      <!-- kinematics -->
-      <wheel_separation>0.1625</wheel_separation>
-      <wheel_diameter>0.06</wheel_diameter>
-      <!-- limits -->
-      <max_wheel_torque>1.0</max_wheel_torque>
-      <max_wheel_acceleration>1.0</max_wheel_acceleration>
-      <!-- output -->
-      <publish_odom>true</publish_odom>
-      <publish_odom_tf>true</publish_odom_tf>
-      <odometry_frame>odom</odometry_frame>
-      <robot_base_frame>base_link</robot_base_frame>
+        <ros>
+            <namespace>/${robot_name}</namespace>
+            <remapping>/cmd_vel:=cmd_vel</remapping>
+        </ros>
+        <!-- wheels -->
+        <left_joint>joint_left_wheel</left_joint>
+        <right_joint>joint_right_wheel</right_joint>
+        <!-- kinematics -->
+        <wheel_separation>0.1625</wheel_separation>
+        <wheel_diameter>0.06</wheel_diameter>
+        <!-- limits -->
+        <max_wheel_torque>1.0</max_wheel_torque>
+        <max_wheel_acceleration>1.0</max_wheel_acceleration>
+        <!-- output -->
+        <publish_odom>true</publish_odom>
+        <publish_odom_tf>true</publish_odom_tf>
+        <odometry_frame>${robot_name}/odom</odometry_frame>>
+        <robot_base_frame>${robot_name}/base_link</robot_base_frame>
     </plugin>
   </gazebo>
@@ -256,5 +269,5 @@
                 <plugin name="laser" filename="libgazebo_ros_ray_sensor.so">
                 <ros>
-                    <namespace>/Morty</namespace>
+                    <namespace>/${robot_name}</namespace>
                     <remapping>~/out:=scan</remapping>
                 </ros>

Commit message: part2

File: xacro/barista_robot_model.urdf.xacro (robot description, xacro)
@@ -29,5 +29,5 @@
 <xacro:property name="sensor_mass"   value="0.300"/>
 <xacro:property name="mesh_path"     value="file://$(find barista_robot_description)/meshes/rplidar_a2.dae"/>
-<xacro:property name="include_laser" value="false"/>
+<xacro:property name="include_laser" value="true"/>
 <!-- Base link  -->
     <link name="base_link">
@@ -256,5 +256,4 @@
                 <plugin name="laser" filename="libgazebo_ros_ray_sensor.so">
                 <ros>
-                    <namespace>/Morty</namespace>
                     <remapping>~/out:=scan</remapping>
                 </ros>

Commit message: ready

File: xacro/barista_robot_model.urdf.xacro (robot description, xacro)
@@ -30,5 +30,5 @@
 <xacro:property name="sensor_mass"   value="0.300"/>
 <xacro:property name="mesh_path"     value="file://$(find barista_robot_description)/meshes/rplidar_a2.dae"/>
-<xacro:property name="include_laser" value="false"/>
+<xacro:property name="include_laser" value="true"/>
   <link name="base_footprint">
   </link>

Commit message: both robots-1-Rviz/gazebo_good/problem with frame world with 1 robot

File: xacro/barista_robot_model.urdf.xacro (robot description, xacro)
@@ -31,6 +31,6 @@
 <xacro:property name="mesh_path"     value="file://$(find barista_robot_description)/meshes/rplidar_a2.dae"/>
 <xacro:property name="include_laser" value="true"/>
-  <link name="base_footprint">
-  </link>
+  <!-- <link name="base_footprint">
+  </link> -->
 <!-- Base link  -->
     <link name="base_link">
@@ -53,9 +53,9 @@
         </inertial>
     </link>
-  <joint name="base_link_joint" type="fixed">
+  <!-- <joint name="base_link_joint" type="fixed">
     <origin rpy="0 0 0" xyz="0 0 0" />
     <parent link="base_footprint" />
     <child link="base_link" />
-  </joint>
+  </joint> -->
   <!-- Wheel Left -->
  <xacro:wheel  wheel_name="left_wheel"        wheel_length=  "${wheel_length}"
